File: ADF5355_Board/MCU.kicad_sch (KiCad schematic)
At the start: 34 parts, among them SW1 SW_SPDT, SW2 SW_Push, U2 STM32L433CCTx, Y1 8MHz, Y2 32kHz

Commit message: Split the project in two
Split the main project in two parts
One is the MCU part and the second is VCO
This was made for the purpose of designing two PCB boards.
In case the MCU part is not designed properly, it can be remade on a cheaper material than the VCO board.
Parts:
- SW1: footprint (none) -> ADF5355:Toggle_switch_710X
- SW2: footprint (none) -> ADF5355:WS_TASV_SMT_Switch
- Y1: footprint (none) -> ADF5355:NX3225GD
